Commit message: Inverted the laser for convenience with poseslam

File: reem_description/urdf/base/base.urdf.xacro (robot description, xacro)
@@ -231,5 +231,5 @@
    <!-- base laser -->
     <xacro:sick_reem_laser name="${name}_laser" parent="${name}" ros_topic="scan_filtered" update_rate="25" min_angle="${-79 * deg_to_rad}" max_angle="${79 * deg_to_rad}" >
-      <origin xyz="${base_laser_x} ${base_laser_y} ${base_laser_z}" rpy="${180.0 * deg_to_rad} 0 0" />
+      <origin xyz="${base_laser_x} ${base_laser_y} ${base_laser_z}" rpy="${0.0 * deg_to_rad} 0 0" />
     </xacro:sick_reem_laser>
    <!-- torso laser -->
